Commit message: First working commit

File: panda_description/urdf/panda.urdf (robot description, URDF)
Before this commit: robot panda, 14 links, 13 joints
Links:
- added link panda_leftfingertip, mass 1e-5
- added link panda_rightfingertip, mass 1e-5
Joints:
- added joint panda_leftfingertip_virtual_joint: type fixed, parent panda_leftfinger, child panda_leftfingertip, origin xyz=0 0 0.045 rpy=0 0 0
- added joint panda_rightfingertip_virtual_joint: type fixed, parent panda_rightfinger, child panda_rightfingertip, origin xyz=0 0 0.045 rpy=0 0 0

File: panda_description/urdf/panda.urdf.xacro (robot description, xacro)
@@ -39,5 +39,5 @@
   <xacro:arg name="ros2_controller_parameters" default="$(find panda_moveit_config)/config/controllers_$(arg ros2_control_command_interface).yaml"/>
   <!-- Flag to preserve fixed joints and prevent lumping when generating SDF for Gazebo -->
-  <xacro:arg name="gazebo_preserve_fixed_joint" default="false"/>
+  <xacro:arg name="gazebo_preserve_fixed_joint" default="true"/>
   <!--            -->
   <!-- Properties -->

File: panda_description/urdf/panda_utils.xacro (robot description, xacro)
@@ -68,4 +68,5 @@
     gazebo_spring_reference:=0.0
     gazebo_preserve_fixed_joint:=false
+    gazebo_add_FT_sensor:=false
   ">
     <!-- Make sure limits are set for non-fixed joints -->
@@ -108,4 +109,19 @@
       </xacro:unless>
     </joint>
+    <!-- Force Torque sensor in each joint -->
+    <xacro:if value="${gazebo_add_FT_sensor}">
+      <gazebo reference="${joint_name}">
+        <sensor name="${joint_name}_FT" type="force_torque">
+          <always_on>true</always_on>
+          <update_rate>20.0</update_rate>
+          <visualize>true</visualize>
+          <topic>${joint_name}_FT</topic>
+          <force_torque>
+            <frame>sensor</frame>
+            <measure_direction>parent_to_child</measure_direction>
+          </force_torque>
+        </sensor>
+      </gazebo>
+    </xacro:if>
     <!-- Transmission for non-fixed joints -->
     <xacro:unless value="${joint_type == 'fixed'}">
@@ -131,5 +147,5 @@
       <gazebo reference="${joint_name}">
         <preserveFixedJoint>true</preserveFixedJoint>
-        <disableFixedJointLumping>true</disableFixedJointLumping>
+        <!--<disableFixedJointLumping>true</disableFixedJointLumping>-->
       </gazebo>
     </xacro:if>
@@ -144,4 +160,5 @@
     joint_origin_rpy
     gazebo_preserve_fixed_joint:=false
+    gazebo_add_FT_sensor:=false
   ">
     <xacro:panda_dummy_link
@@ -154,4 +171,18 @@
       <origin xyz="${joint_origin_xyz}" rpy="${joint_origin_rpy}"/>
     </joint>
+    <xacro:if value="${gazebo_add_FT_sensor}">
+      <gazebo reference="${link_name}_virtual_joint">
+        <sensor name="${link_name}_FT" type="force_torque">
+          <always_on>true</always_on>
+          <update_rate>20.0</update_rate>
+          <visualize>true</visualize>
+          <topic>${link_name}_FT</topic>
+          <force_torque>
+            <frame>sensor</frame>
+            <measure_direction>parent_to_child</measure_direction>
+          </force_torque>
+        </sensor>
+      </gazebo>
+    </xacro:if>
   </xacro:macro>
   <!--       -->
@@ -174,5 +205,5 @@
       <gazebo reference="${link_name}_virtual_joint">
         <preserveFixedJoint>true</preserveFixedJoint>
-        <disableFixedJointLumping>true</disableFixedJointLumping>
+        <!--<disableFixedJointLumping>true</disableFixedJointLumping>-->
       </gazebo>
     </xacro:if>

File: panda_moveit_config/srdf/panda_gripper.xacro (robot description, xacro)
@@ -12,6 +12,10 @@
       <link name="${prefix}leftfinger"/>
       <link name="${prefix}rightfinger"/>
+      <link name="${prefix}rightfingertip"/>
+      <link name="${prefix}leftfingertip"/>
       <joint name="${prefix}finger_joint1"/>
       <joint name="${prefix}finger_joint2"/>
+      <joint name="${prefix}rightfingertip_virtual_joint"/>
+      <joint name="${prefix}leftfingertip_virtual_joint"/>
     </group>
     <group_state name="open" group="gripper">
@@ -26,4 +30,5 @@
     <disable_collisions link1="${prefix}hand" link2="${prefix}rightfinger" reason="Adjacent"/>
     <disable_collisions link1="${prefix}leftfinger" link2="${prefix}rightfinger" reason="Default"/>
+    <disable_collisions link1="${prefix}leftfingertip" link2="${prefix}rightfingertip" reason="Default"/>
   </xacro:macro>
 </robot>

Commit message: Added Moveit Task Constructor execution in Ignition Gazebo

File: panda_description/urdf/panda.urdf (robot description, URDF)
Before this commit: robot panda, 16 links, 15 joints
Links:
- link panda_hand_tcp: mass None -> 1e-5
- link panda_link8: mass None -> 1e-5
- link world: mass None -> 1e-5

File: panda_description/urdf/panda.urdf.xacro (robot description, xacro)
@@ -35,5 +35,5 @@
   <xacro:arg name="ros2_control_plugin" default="ign"/>
   <!-- The output control command interface provided by ros2_control ('position', 'velocity', 'effort' or certain combinations 'position,velocity') -->
-  <xacro:arg name="ros2_control_command_interface" default="effort"/>
+  <xacro:arg name="ros2_control_command_interface" default="position"/>
   <!-- The filepath to parameters of ROS 2 controllers -->
   <xacro:arg name="ros2_controller_parameters" default="$(find panda_moveit_config)/config/controllers_$(arg ros2_control_command_interface).yaml"/>

File: panda_description/urdf/panda_utils.xacro (robot description, xacro)
@@ -114,5 +114,5 @@
         <sensor name="${joint_name}_FT" type="force_torque">
           <always_on>true</always_on>
-          <update_rate>20.0</update_rate>
+          <update_rate>100.0</update_rate>
           <visualize>true</visualize>
           <topic>${joint_name}_FT</topic>
@@ -175,5 +175,5 @@
         <sensor name="${link_name}_FT" type="force_torque">
           <always_on>true</always_on>
-          <update_rate>20.0</update_rate>
+          <update_rate>100.0</update_rate>
           <visualize>true</visualize>
           <topic>${link_name}_FT</topic>

File: panda_moveit_config/srdf/panda.srdf.xacro (robot description, xacro)
@@ -29,4 +29,9 @@
     prefix="${prefix_gripper}"
   />
+  <!--SUBGROUPS Groups can also be formed by referencing to already defined group names-->
+  <group name="panda_arm_hand">
+    <group name="arm"/>
+    <group name="gripper"/>
+  </group>
   <end_effector group="gripper" name="gripper" parent_group="arm" parent_link="${prefix_arm}hand_tcp"/>
   <disable_collisions link1="${prefix_gripper}hand" link2="${prefix_arm}link3" reason="Never"/>
